Commit message: Updated gifs

File: scara_description/urdf/scara.xacro (robot description, xacro)
@@ -45,5 +45,5 @@
           <box size="${W} ${W} ${L1}"/>
       </geometry>
-      <material name="orange"/>
+      <material name="white"/>
     </visual>
     <inertial>
@@ -75,5 +75,5 @@
           <box size="${W} ${W} ${L2}"/>
       </geometry>
-      <material name="orange"/>
+      <material name="white"/>
     </visual>
     <inertial>
@@ -108,5 +108,5 @@
           <box size="${W} ${W} ${L3}"/>
       </geometry>
-      <material name="orange"/>
+      <material name="white"/>
     </visual>
     <inertial>
@@ -142,5 +142,5 @@
           <box size="${W} ${W} ${L4}"/>
       </geometry>
-      <material name="orange"/>
+      <material name="white"/>
     </visual>
     <inertial>
